File: PID_Vis_PCB + Arduino V2/_autosave-PID_Vis_PCB + Arduino.kicad_pcb (KiCad board)
At the start: 2 copper layers, 126 x 83.8 mm, 31 parts, among them J1 Raspberry_Pi_2_3, J10 Conn_01x04_Male, J11 Conn_01x06_Male, J12 Conn_01x03_Male, J13 Conn_01x02_Male, J14 Conn_01x03_Male, J15 Conn_01x03_Male, J2 Conn_01x04_Male, J3 Conn_01x04_Male, J4 Conn_01x04_Male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

Commit message: Einhverjar breitingar
Parts:
- C1, C2: footprint Capacitor_THT:C_Axial_L3.8mm_D2.6mm_P7.50mm_Horizontal -> Capacitor_THT:C_Disc_D5.0mm_W2.5mm_P2.50mm
- K1: footprint Relay_THT:Relay_SPDT_Finder_36.11 -> Custom:Relay_SRA-05VDC-CL
- moved R8 105.3 mm to (171.2, 72.1)
- moved R9 91.6 mm to (155.4, 80.8), turned to -90 degrees
- moved R5 73.0 mm to (193.8, 79.8)
- moved R4 71.2 mm to (195.6, 83.1)
- moved R7 68.5 mm to (243.8, 89.2)
- moved R6 64.3 mm to (243.8, 86.1)
- moved C1 62.3 mm to (240.3, 86.1), turned to 180 degrees
- moved C2 61.2 mm to (240.3, 89.2), turned to 180 degrees
- moved R3 9.02 mm to (195.1, 68.3), turned to 180 degrees
- moved A1 9.00 mm to (212.2, 98.4)
- moved A2 9.00 mm to (212.2, 118.5)
- moved J2 5.95 mm to (196.3, 117.1), turned to -90 degrees
- moved J11 5.77 mm to (164.8, 92.7), turned to 180 degrees
- moved J1 3.05 mm to (142.7, 104.9)
- moved R1 2.31 mm to (219.6, 70.9)
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Connections:
- A1 pad 10: Net-(A1-Pad10) -> unconnected-(A1-Pad10)
- A2 pad 5: Net-(A2-Pad5) -> Net-(J12-Pad3)
- A2 pad 6: Net-(A2-Pad6) -> Net-(U1-Pad9)
- A2 pad 7: unconnected-(A2-Pad7) -> Net-(U1-Pad10)
- J12 pad 3: Net-(A1-Pad10) -> Net-(J12-Pad3)
- J13 pad 2: Net-(A1-Pad10) -> Net-(J12-Pad3)
- R3 pad 2: Net-(A1-Pad10) -> Net-(J12-Pad3)
- U1 pad 10: Net-(A2-Pad6) -> Net-(U1-Pad10)
- U1 pad 9: Net-(A2-Pad5) -> Net-(U1-Pad9)
- U2 pad 3: Net-(A1-Pad9) -> Net-(A1-Pad8)
- U2 pad 4: Net-(A1-Pad8) -> Net-(A1-Pad9)
Routing:
- net +5V: track 128.8 -> 319.8 mm
- net Net-(A1-Pad15): track 0.00 -> 148.6 mm, vias 0 -> 1
- net +3.3V: track 28.9 -> 130.1 mm, vias 0 -> 2
- net Net-(J12-Pad3): track 0.00 -> 92.5 mm
- net Net-(J1-Pad13): track 0.00 -> 89.7 mm, vias 0 -> 2
- net Net-(A1-Pad12): track 8.73 -> 91.2 mm, vias 0 -> 1
- net Net-(A1-Pad11): track 10.5 -> 89.6 mm, vias 0 -> 2
- net Net-(J1-Pad15): track 0.00 -> 78.1 mm, vias 0 -> 2
- net Net-(R4-Pad2): track 0.00 -> 68.8 mm
- net Net-(R5-Pad2): track 0.00 -> 68.3 mm
- net Net-(U1-Pad10): track 0.00 -> 63.5 mm
- net Net-(U1-Pad9): track 0.00 -> 62.9 mm
- net Net-(J1-Pad12): track 0.00 -> 61.8 mm
- net Net-(J1-Pad5): track 0.00 -> 56.2 mm, vias 0 -> 2
- net Net-(J1-Pad3): track 0.00 -> 56.2 mm, vias 0 -> 2
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Other:
- board text added: "+3.3V"
- board text added: "3.3V SIG"
- board text added: "5V SIG"
- board text added: "A1"
- board text added: "Endastopp DC"
- board text added: "I2C"
