File: PID_Vis_PCB + Arduino V2/PID_Vis_PCB + Arduino.kicad_pcb (KiCad board)
At the start: 2 copper layers, 126 x 83.8 mm, 26 parts, among them J1 Raspberry_Pi_2_3, J10 Conn_01x04_Male, J11 Conn_01x06_Male, J12 Conn_01x03_Male, J13 Conn_01x02_Male, J2 Conn_01x04_Male, J3 Conn_01x04_Male, J4 Conn_01x04_Male, J5 Conn_01x06_Male, J6 Conn_01x03_Male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

Commit message: Einhverjar breitingar
Parts:
- added J14: Conn_01x03_Male, Connector_Phoenix_MC:PhoenixContact_MC_1,5_3-G-3.5_1x03_P3.50mm_Horizontal, F.Cu at (166.9, 49.3)
- added J15: Conn_01x03_Male, Connector_Phoenix_MC:PhoenixContact_MC_1,5_3-G-3.5_1x03_P3.50mm_Horizontal, F.Cu at (180.0, 49.3)
- added K1: FINDER-36.11, Custom:Relay_SRA-05VDC-CL, F.Cu at (167.9, 66.6)
- added R8: 10k, Resistor_THT:R_Axial_DIN0207_L6.3mm_D2.5mm_P10.16mm_Horizontal, F.Cu at (171.2, 72.1)
- added R9: 10k, Resistor_THT:R_Axial_DIN0207_L6.3mm_D2.5mm_P10.16mm_Horizontal, F.Cu at (155.4, 80.8)
- moved U1 100.7 mm to (218.3, 69.3), turned to -90 degrees
- moved R5 73.0 mm to (193.8, 79.8)
- moved R4 71.2 mm to (195.6, 83.1)
- moved R7 68.5 mm to (243.8, 89.2)
- moved R6 64.3 mm to (243.8, 86.1)
- moved C1 62.3 mm to (240.3, 86.1), turned to 180 degrees
- moved C2 61.2 mm to (240.3, 89.2), turned to 180 degrees
- moved J3 48.8 mm to (209.7, 49.3)
- moved J4 48.0 mm to (208.2, 55.0)
- moved J9 30.0 mm to (226.3, 49.3)
- moved J10 28.5 mm to (223.9, 54.9)
- moved R2 28.5 mm to (216.2, 69.3)
- moved R1 26.8 mm to (219.6, 70.9)
- moved R3 22.6 mm to (195.1, 68.3), turned to 180 degrees
- moved J12 13.7 mm to (193.0, 49.3)
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Connections:
- A1 pad 10: Net-(A1-Pad10) -> unconnected-(A1-Pad10)
- A1 pad 15: unconnected-(A1-Pad15) -> Net-(A1-Pad15)
- A2 pad 15: unconnected-(A2-Pad15) -> Net-(A1-Pad15)
- A2 pad 5: Net-(A2-Pad5) -> Net-(J12-Pad3)
- A2 pad 6: Net-(A2-Pad6) -> Net-(U1-Pad9)
- A2 pad 7: unconnected-(A2-Pad7) -> Net-(U1-Pad10)
- J1 pad 12: unconnected-(J1-Pad12) -> Net-(J1-Pad12)
- J12 pad 3: Net-(A1-Pad10) -> Net-(J12-Pad3)
- J13 pad 2: Net-(A1-Pad10) -> Net-(J12-Pad3)
- J8 pad 1: +12V -> Net-(J8-Pad1)
- R3 pad 2: Net-(A1-Pad10) -> Net-(J12-Pad3)
- U1 pad 10: Net-(A2-Pad6) -> Net-(U1-Pad10)
- U1 pad 9: Net-(A2-Pad5) -> Net-(U1-Pad9)
- U2 pad 3: Net-(A1-Pad9) -> Net-(A1-Pad8)
- U2 pad 4: Net-(A1-Pad8) -> Net-(A1-Pad9)
Routing:
- net Net-(A1-Pad15): track 0.00 -> 148.3 mm, vias 0 -> 1
- net +5V: track 200.7 -> 318.6 mm
- net Net-(J12-Pad3): track 0.00 -> 91.6 mm
- net Net-(J1-Pad13): track 0.00 -> 89.7 mm, vias 0 -> 2
- net +3.3V: track 42.3 -> 130.1 mm, vias 0 -> 2
- net Net-(A1-Pad12): track 10.7 -> 92.4 mm, vias 0 -> 1
- net Net-(A1-Pad11): track 9.93 -> 89.6 mm, vias 0 -> 2
- net Net-(J1-Pad15): track 0.00 -> 76.3 mm, vias 0 -> 2
- net Net-(R4-Pad2): track 0.00 -> 67.7 mm
- net Net-(R5-Pad2): track 0.00 -> 67.6 mm
- net Net-(U1-Pad10): track 0.00 -> 62.6 mm
- net Net-(U1-Pad9): track 0.00 -> 62.0 mm
- net Net-(J1-Pad12): track 0.00 -> 61.8 mm
- net Net-(J1-Pad5): track 0.00 -> 56.2 mm, vias 0 -> 2
- net Net-(J1-Pad3): track 0.00 -> 56.2 mm, vias 0 -> 2
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- removed copper zone on F.Cu, net GND
Other:
- outline, holes or cut-outs redrawn

Commit message: stuff
Parts:
- C1, C2: footprint Capacitor_THT:C_Axial_L3.8mm_D2.6mm_P7.50mm_Horizontal -> Capacitor_THT:C_Disc_D5.0mm_W2.5mm_P2.50mm
- moved R4 4.64 mm to (191.0, 82.3)
- moved R5 0.92 mm to (193.0, 79.2)
Connections:
- A2 pad 10: Net-(R4-Pad2) -> Net-(A2-Pad10)
- A2 pad 6: Net-(U1-Pad9) -> Net-(R4-Pad2)
- A2 pad 7: Net-(U1-Pad10) -> Net-(R5-Pad2)
- A2 pad 9: Net-(R5-Pad2) -> Net-(A2-Pad9)
- J3 pad 1: Net-(J3-Pad1) -> Net-(U1-Pad6)
- J3 pad 2: Net-(J3-Pad2) -> Net-(U1-Pad5)
- J3 pad 3: Net-(J3-Pad3) -> Net-(U1-Pad4)
- J3 pad 4: Net-(J3-Pad4) -> Net-(U1-Pad3)
- J4 pad 1: Net-(J3-Pad1) -> Net-(U1-Pad6)
- J4 pad 2: Net-(J3-Pad2) -> Net-(U1-Pad5)
- J4 pad 3: Net-(J3-Pad3) -> Net-(U1-Pad4)
- J4 pad 4: Net-(J3-Pad4) -> Net-(U1-Pad3)
- K1 pad 12: GND -> unconnected-(K1-Pad12)
- U1 pad 10: Net-(U1-Pad10) -> Net-(A2-Pad9)
- U1 pad 3: Net-(J3-Pad1) -> Net-(U1-Pad3)
- U1 pad 4: Net-(J3-Pad2) -> Net-(U1-Pad4)
- U1 pad 5: Net-(J3-Pad3) -> Net-(U1-Pad5)
- U1 pad 6: Net-(J3-Pad4) -> Net-(U1-Pad6)
- U1 pad 9: Net-(U1-Pad9) -> Net-(A2-Pad10)
Routing:
- net Net-(A2-Pad10): track 0.00 -> 68.8 mm
- net Net-(A2-Pad9): track 0.00 -> 67.7 mm
- net Net-(U1-Pad10): track 62.6 -> 0.00 mm
- net Net-(U1-Pad9): track 62.0 -> 0.00 mm
- net Net-(U1-Pad6): track 0.00 -> 14.3 mm
- net Net-(J3-Pad1): track 14.3 -> 0.00 mm
- net Net-(U1-Pad3): track 0.00 -> 14.3 mm
- net Net-(J3-Pad4): track 14.3 -> 0.00 mm
- net Net-(U1-Pad5): track 0.00 -> 13.9 mm
- net Net-(J3-Pad2): track 13.9 -> 0.00 mm
- net Net-(U1-Pad4): track 0.00 -> 13.9 mm
- net Net-(J3-Pad3): track 13.9 -> 0.00 mm
- net Net-(R4-Pad2): track 67.7 -> 62.2 mm
- net Net-(R5-Pad2): track 67.6 -> 63.1 mm
- net +12V: track 126.9 -> 130.1 mm
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- added copper zone on F.Cu, net GND
Other:
- board size 126 x 83.8 mm -> 124 x 83.8 mm
- board text added: "+3.3V"
- board text added: "3.3V SIG"
- board text added: "5V SIG"
- board text added: "A1"
- board text added: "Endastopp DC"
- board text added: "I2C"
