File: PID_Vis_PCB + Arduino V2/PID_Vis_PCB + Arduino.kicad_pcb (KiCad board)
At the start: 2 copper layers, 126 x 83.8 mm, 31 parts, among them J1 Raspberry_Pi_2_3, J10 Conn_01x04_Male, J11 Conn_01x06_Male, J12 Conn_01x03_Male, J13 Conn_01x02_Male, J14 Conn_01x03_Male, J15 Conn_01x03_Male, J2 Conn_01x04_Male, J3 Conn_01x04_Male, J4 Conn_01x04_Male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

Commit message: Schematic change
Parts:
- C1, C2: footprint Capacitor_THT:C_Axial_L3.8mm_D2.6mm_P7.50mm_Horizontal -> Capacitor_THT:C_Disc_D5.0mm_W2.5mm_P2.50mm
- moved R4 4.64 mm to (191.0, 82.3)
- moved R5 0.92 mm to (193.0, 79.2)
Connections:
- A2 pad 10: Net-(R4-Pad2) -> Net-(A2-Pad10)
- A2 pad 6: Net-(U1-Pad9) -> Net-(R4-Pad2)
- A2 pad 7: Net-(U1-Pad10) -> Net-(R5-Pad2)
- A2 pad 9: Net-(R5-Pad2) -> Net-(A2-Pad9)
- J3 pad 1: Net-(J3-Pad1) -> Net-(U1-Pad6)
- J3 pad 2: Net-(J3-Pad2) -> Net-(U1-Pad5)
- J3 pad 3: Net-(J3-Pad3) -> Net-(U1-Pad4)
- J3 pad 4: Net-(J3-Pad4) -> Net-(U1-Pad3)
- J4 pad 1: Net-(J3-Pad1) -> Net-(U1-Pad6)
- J4 pad 2: Net-(J3-Pad2) -> Net-(U1-Pad5)
- J4 pad 3: Net-(J3-Pad3) -> Net-(U1-Pad4)
- J4 pad 4: Net-(J3-Pad4) -> Net-(U1-Pad3)
- K1 pad 12: GND -> unconnected-(K1-Pad12)
- U1 pad 10: Net-(U1-Pad10) -> Net-(A2-Pad9)
- U1 pad 3: Net-(J3-Pad1) -> Net-(U1-Pad3)
- U1 pad 4: Net-(J3-Pad2) -> Net-(U1-Pad4)
- U1 pad 5: Net-(J3-Pad3) -> Net-(U1-Pad5)
- U1 pad 6: Net-(J3-Pad4) -> Net-(U1-Pad6)
- U1 pad 9: Net-(U1-Pad9) -> Net-(A2-Pad10)
Routing:
- net Net-(A2-Pad10): track 0.00 -> 68.8 mm
- net Net-(A2-Pad9): track 0.00 -> 67.7 mm
- net Net-(U1-Pad10): track 62.6 -> 0.00 mm
- net Net-(U1-Pad9): track 62.0 -> 0.00 mm
- net Net-(U1-Pad6): track 0.00 -> 14.3 mm
- net Net-(J3-Pad1): track 14.3 -> 0.00 mm
- net Net-(U1-Pad3): track 0.00 -> 14.3 mm
- net Net-(J3-Pad4): track 14.3 -> 0.00 mm
- net Net-(U1-Pad5): track 0.00 -> 13.9 mm
- net Net-(J3-Pad2): track 13.9 -> 0.00 mm
- net Net-(U1-Pad4): track 0.00 -> 13.9 mm
- net Net-(J3-Pad3): track 13.9 -> 0.00 mm
- net Net-(R4-Pad2): track 67.7 -> 62.2 mm
- net Net-(R5-Pad2): track 67.6 -> 63.1 mm
- net +12V: track 126.9 -> 130.1 mm
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- added copper zone on F.Cu, net GND
Other:
- board size 126 x 83.8 mm -> 124 x 83.8 mm
- board text added: "+3.3V"
- board text added: "3.3V SIG"
- board text added: "5V SIG"
- board text added: "A1"
- board text added: "Endastopp DC"
- board text added: "I2C"
