File: PID_Vis_PCB + Arduino V2/_autosave-PID_Vis_PCB + Arduino.kicad_sch (KiCad schematic)
At the start: 31 parts, among them J1 Raspberry_Pi_2_3, J10 Conn_01x04_Male, J11 Conn_01x06_Male, J12 Conn_01x03_Male, J13 Conn_01x02_Male, J14 Conn_01x03_Male, J15 Conn_01x03_Male, J2 Conn_01x04_Male, J3 Conn_01x04_Male, J4 Conn_01x04_Male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

Commit message: stuff
Connections:
- net GND: no longer K1.12
- net at R4.2, U1.15 (MS1): now also A2.6 (D3); no longer A2.10 (D7)
- net at U1.9 (DIR): now also A2.10 (D7); no longer A2.6 (D3)
- net at A2.7 (D4): now also R5.2, U1.14 (MS2); no longer U1.10 (STEP)
- net at J3.1 (Pin_1), J4.1 (Pin_1): now also U1.6 (M2B); no longer U1.3 (M1B)
- net at J3.2 (Pin_2), J4.2 (Pin_2): now also U1.5 (M2A); no longer U1.4 (M1A)
- net at J3.3 (Pin_3), J4.3 (Pin_3): now also U1.4 (M1A); no longer U1.5 (M2A)
- net at J3.4 (Pin_4), J4.4 (Pin_4): now also U1.3 (M1B); no longer U1.6 (M2B)
- new net: A2.9 (D6), U1.10 (STEP)
Other:
- moved on the sheet: J3, J4
