File: PID_Vis_PCB + Arduino V3/PID_Vis_PCB + Arduino.kicad_sch (KiCad schematic)
At the start: 31 parts, among them J1 Raspberry_Pi_2_3, J10 Conn_01x04_Male, J11 Conn_01x06_Male, J12 Conn_01x03_Male, J13 Conn_01x02_Male, J14 Conn_01x03_Male, J15 Conn_01x03_Male, J2 Conn_01x04_Male, J3 Conn_01x04_Male, J4 Conn_01x04_Male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

Commit message: Schematic change
Connections:
- net +5V: now also U2.1 (VM)
- net 5V Estop signal: no longer names the net of A1.15 (D12), A2.15 (D12), J15.1 (Pin_1), R8.2
Other:
- note removed: "Estop Connector"
- note removed: "I2C Connector"
- moved on the sheet: C1, C2, J1, J10, J11, J12, J13, J2, J3, J4, J5, J6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
